File: _autosave-Batteryboard.sch (KiCad schematic (older format))
At the start: 95 parts, among them J1 Conn_01x02_Male, J2 Conn_01x03_Male, J3 Conn_01x02_Male, J4 Conn_01x02_Male, J5 SC_19-20, Q1 SI7617DN-T1-GE3, Q2 SI7617DN-T1-GE3, Q3 SI7617DN-T1-GE3, Q4 SIS412DN-T1-GE3, Q5 SIS412DN-T1-GE3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

Commit message: first commit, still have a way to go
Parts:
- added C? (x6): C, symbol Device:C
- added L?: 4.7uH, symbol Device:L
- added R? (x5): R_US, symbol Device:R_US
Connections:
- net 3V3: now also C?.2, C?.2, L?.2, R?.2
- net 5V0: now also TMP1.1 (Vs), C?.2, C?.2, L?.1, R?.2
- net FB1: now also C?.1, R?.1, R?.2
- net GND: now also TMP1.3 (GND), U2.23 (AGND), U2.37 (EPAD), C?.1, C?.1, C?.1, C?.1, C?.1, R?.1, R?.1
- net LX1: now also L?.2
- net RLIM2: now also U2.30 (VOUT2); no longer U2.31 (RLIM2)
- net TEMP_OUT: now reaches TMP1.2 (Vout)
- net at U2.20 (SS1): now also C?.2
- net at U2.21 (COMP1): now also R?.2
- net at U2.22 (ROSC): now also R?.2
- net at U2.24 (COMP2): now also R?.2
- net at U2.25 (SS2): now also C?.2
- net FB2: no longer names the net of C?.1, R?.1, R?.2
- net FB2: now also U2.31 (RLIM2)
- new net: C?.2, R?.1 (x2)
Other:
- moved on the sheet: J5, TMP1
