File: Batteryboard.sch (KiCad schematic (older format))
At the start: 148 parts, among them IC1 FAN4010IL6X_F113, IC2 FAN4010IL6X_F113, IC3 FAN4010IL6X_F113, J1 Conn_01x02_Male, J2 Conn_01x03_Male, J3 Conn_01x05_Male, J4 Conn_01x02_Male, J5 SC_19-20, Q1 SI7617DN-T1-GE3, Q2 SI7617DN-T1-GE3, Q3 SI7617DN-T1-GE3, Q4 SIS412DN-T1-GE3, Q5 SIS412DN-T1-GE3, Q6 SIS412DN-T1-GE3, Q7 SI7617DN-T1-GE3, Q8 SIS412DN-T1-GE3, U1 BQ24617RGET, U2 TPS65279DAPR, U3 BQ29200DRBT, U4 PIC18F25K50-I_SO, U5 MCP2515-xSO, U6 SN65HVD1050D

Commit message: big overhaul on board, did a bunch of stuff
Parts:
- C20, C21, C34, C35, C38, C50: value C -> .1uF
- C26, C27: value C -> 50nF
- R10, R32, R9: value R_US -> 10kOhm
- R21, R22: value R_US -> 60.4kOhm
- R28: value R_US -> 30Ohm
- R33: value R_US -> 470Ohm
- R44, R45: value R_US -> 100Ohm
Connections:
- net GND: no longer C12.2, C13.2, C16.2, C18.1, C19.2, C22.2, C23.1, C31.1, C44.1, C45.1, C46.1, C47.1, C48.1, C49.1, C5.2, C8.2, C9.2, CCD1.2, CIN2.2, CVD1.2, J1.2 (Pin_2), J2.3 (Pin_3), J4.1 (Pin_1), Q5.1 (S_1), Q5.2 (S_2), Q5.3 (S_3), Q7.5 (D_1), Q7.6 (D_2), Q7.7 (D_3), Q7.8 (D_4), Q8.1 (S_1), Q8.2 (S_2), Q8.3 (S_3), R10.2, R_JUMP1.2, U1.17 (GND), U2.10 (PGND1), U2.11 (PGND1), U2.34 (PGND2), U2.35 (PGND2), U2.36 (PGND2), U2.37 (EPAD), U2.9 (PGND1), U3.5 (GND), U3.6 (*CB_EN), U3.9 (EPAD)
- new net GNDREF: C12.2, C13.2, C16.2, C18.1, C19.2, C22.2, C23.1, C31.1, C44.1, C45.1, C46.1, C47.1, C48.1, C49.1, C5.2, C8.2, C9.2, CCD1.2, CIN2.2, CVD1.2, J1.2 (Pin_2), J2.3 (Pin_3), J4.1 (Pin_1), Q5.1 (S_1), Q5.2 (S_2), Q5.3 (S_3), Q7.5 (D_1), Q7.6 (D_2), Q7.7 (D_3), Q7.8 (D_4), Q8.1 (S_1), Q8.2 (S_2), Q8.3 (S_3), R10.2, R_JUMP1.2, U1.17 (GND), U2.10 (PGND1), U2.11 (PGND1), U2.34 (PGND2), U2.35 (PGND2), U2.36 (PGND2), U2.37 (EPAD), U2.9 (PGND1), U3.5 (GND), U3.6 (*CB_EN), U3.9 (EPAD)
Other:
- moved on the sheet: C38
Changed lines of the file:
@@
 Wire Wire Line
 	7050 5050 7050 4500
-Wire Wire Line
-	7050 4500 6900 4500
 Connection ~ 7450 5050
 Wire Wire Line
@@
 	0    1    1    0
 $EndComp
-$Comp
-L power:GND #PWR0107
-U 1 1 5DBBAFAE
-P 6900 4550
-F 0 "#PWR0107" H 6900 4300 50  0001 C CNN
-F 1 "GND" H 6905 4377 50  0000 C CNN
-F 2 "" H 6900 4550 50  0001 C CNN
-F 3 "" H 6900 4550 50  0001 C CNN
-	1    6900 4550
-	1    0    0    -1
-$EndComp
-Wire Wire Line
-	6900 4550 6900 4500
 Wire Wire Line
 	6300 5300 6500 5300
@@
 Text GLabel 8000 5150 3    50   Input ~ 0
 SRP
-Connection ~ 6900 4500
 Text GLabel 8350 5150 3    50   Input ~ 0
 SRN
@@
 	1500 5250 1500 5600
 Wire Wire Line
-	6450 4500 6900 4500
-Wire Wire Line
 	7150 4300 6450 4300
 Wire Wire Line
@@
 Wire Wire Line
 	16400 3450 16400 4000
-Text GLabel 12250 6600 1    50   Input ~ 0
-PGND2
 Text GLabel 8000 9100 2    50   Input ~ 0
 TS
@@
 P 4150 8400
 F 0 "R10" H 4218 8446 50  0000 L CNN
-F 1 "R_US" H 4218 8355 50  0000 L CNN
+F 1 "10kOhm" H 4218 8355 50  0000 L CNN
 F 2 "Resistor_SMD:R_0603_1608Metric" V 4190 8390 50  0001 C CNN
 F 3 "~" H 4150 8400 50  0001 C CNN
@@
 P 4150 8000
 F 0 "R9" H 4218 8046 50  0000 L CNN
-F 1 "R_US" H 4218 7955 50  0000 L CNN
+F 1 "10kOhm" H 4218 7955 50  0000 L CNN
 F 2 "Resistor_SMD:R_0603_1608Metric" V 4190 7990 50  0001 C CNN
 F 3 "~" H 4150 8000 50  0001 C CNN
@@
 P 5000 9450
 F 0 "C34" V 5252 9450 50  0000 C CNN
-F 1 "C" V 5161 9450 50  0000 C CNN
+F 1 ".1uF" V 5161 9450 50  0000 C CNN
 F 2 "Capacitor_SMD:C_0603_1608Metric" H 5038 9300 50  0001 C CNN
 F 3 "~" H 5000 9450 50  0001 C CNN
@@
 P 5250 7100
 F 0 "R32" H 5318 7146 50  0000 L CNN
-F 1 "R_US" H 5318 7055 50  0000 L CNN
+F 1 "10kOhm" H 5318 7055 50  0000 L CNN
 F 2 "Resistor_SMD:R_0603_1608Metric" V 5290 7090 50  0001 C CNN
 F 3 "~" H 5250 7100 50  0001 C CNN
@@
 P 5250 7400
 F 0 "C35" H 5365 7446 50  0000 L CNN
-F 1 "C" H 5365 7355 50  0000 L CNN
+F 1 ".1uF" H 5365 7355 50  0000 L CNN
 F 2 "Capacitor_SMD:C_0603_1608Metric" H 5288 7250 50  0001 C CNN
 F 3 "~" H 5250 7400 50  0001 C CNN
@@
 P 5450 7250
 F 0 "R33" V 5655 7250 50  0000 C CNN
-F 1 "R_US" V 5564 7250 50  0000 C CNN
+F 1 "470Ohm" V 5564 7250 50  0000 C CNN
 F 2 "Resistor_SMD:R_0603_1608Metric" V 5490 7240 50  0001 C CNN
 F 3 "~" H 5450 7250 50  0001 C CNN
@@
 Text GLabel 5000 8000 0    50   Input ~ 0
 MCLR
-Text GLabel 8000 8900 2    50   Input ~ 0
-VSS
 Text GLabel 8000 8800 2    50   Input ~ 0
 VDD
-Text GLabel 6300 6950 0    50   Input ~ 0
+Text GLabel 6300 7000 0    50   Input ~ 0
 5V0
-Text GLabel 6800 6950 2    50   Input ~ 0
+Text GLabel 6800 7000 2    50   Input ~ 0
 VDD
 Text GLabel 1700 12900 2    50   Input ~ 0
@@
 P 13400 9350
 F 0 "C20" V 13148 9350 50  0000 C CNN
-F 1 "C" V 13239 9350 50  0000 C CNN
+F 1 ".1uF" V 13239 9350 50  0000 C CNN
 F 2 "Capacitor_SMD:C_0603_1608Metric" H 13438 9200 50  0001 C CNN
 F 3 "~" H 13400 9350 50  0001 C CNN
@@
 P 14450 8500
 F 0 "R28" V 14245 8500 50  0000 C CNN
-F 1 "R_US" V 14336 8500 50  0000 C CNN
+F 1 "30Ohm" V 14336 8500 50  0000 C CNN
 F 2 "Resistor_SMD:R_0603_1608Metric" V 14490 8490 50  0001 C CNN
 F 3 "~" H 14450 8500 50  0001 C CNN
@@
 P 14450 8700
 F 0 "C27" V 14198 8700 50  0000 C CNN
-F 1 "C" V 14289 8700 50  0000 C CNN
+F 1 "50nF" V 14289 8700 50  0000 C CNN
 F 2 "Capacitor_SMD:C_0603_1608Metric" H 14488 8550 50  0001 C CNN
 F 3 "~" H 14450 8700 50  0001 C CNN
@@
 P 14450 8200
 F 0 "C26" V 14198 8200 50  0000 C CNN
-F 1 "C" V 14289 8200 50  0000 C CNN
+F 1 "50nF" V 14289 8200 50  0000 C CNN
 F 2 "Capacitor_SMD:C_0603_1608Metric" H 14488 8050 50  0001 C CNN
 F 3 "~" H 14450 8200 50  0001 C CNN
@@
 P 13400 9550
 F 0 "R21" V 13195 9550 50  0000 C CNN
-F 1 "R_US" V 13286 9550 50  0000 C CNN
+F 1 "60.4kOhm" V 13286 9550 50  0000 C CNN
 F 2 "Resistor_SMD:R_0603_1608Metric" V 13440 9540 50  0001 C CNN
 F 3 "~" H 13400 9550 50  0001 C CNN
@@
 P 13400 9950
 F 0 "C21" V 13148 9950 50  0000 C CNN
-F 1 "C" V 13239 9950 50  0000 C CNN
+F 1 ".1uF" V 13239 9950 50  0000 C CNN
 F 2 "Capacitor_SMD:C_0603_1608Metric" H 13438 9800 50  0001 C CNN
 F 3 "~" H 13400 9950 50  0001 C CNN
@@
 P 13400 10150
 F 0 "R22" V 13195 10150 50  0000 C CNN
-F 1 "R_US" V 13286 10150 50  0000 C CNN
+F 1 "60.4kOhm" V 13286 10150 50  0000 C CNN
 F 2 "Resistor_SMD:R_0603_1608Metric" V 13440 10140 50  0001 C CNN
 F 3 "~" H 13400 10150 50  0001 C CNN
@@
 Text GLabel 5000 8700 0    50   Input ~ 0
 VSS
-Connection ~ 6550 6950
+Connection ~ 6550 7000
 Wire Wire Line
-	6550 6950 6800 6950
+	6550 7000 6800 7000
 Wire Wire Line
-	6300 6950 6550 6950
+	6300 7000 6550 7000
 Wire Wire Line
 	8000 7150 8000 6900
@@
 P 7600 7150
 F 0 "R45" V 7805 7150 50  0000 C CNN
-F 1 "R_US" V 7714 7150 50  0000 C CNN
+F 1 "100Ohm" V 7714 7150 50  0000 C CNN
 F 2 "Resistor_SMD:R_0603_1608Metric" V 7640 7140 50  0001 C CNN
 F 3 "~" H 7600 7150 50  0001 C CNN
@@
 P 7600 7050
 F 0 "R44" V 7395 7050 50  0000 C CNN
-F 1 "R_US" V 7486 7050 50  0000 C CNN
+F 1 "100Ohm" V 7486 7050 50  0000 C CNN
 F 2 "Resistor_SMD:R_0603_1608Metric" V 7640 7040 50  0001 C CNN
 F 3 "~" H 7600 7050 50  0001 C CNN
@@
 P 8050 7450
 F 0 "C50" V 7798 7450 50  0000 C CNN
-F 1 "C" V 7889 7450 50  0000 C CNN
+F 1 ".1uF" V 7889 7450 50  0000 C CNN
 F 2 "Capacitor_SMD:C_0603_1608Metric" H 8088 7300 50  0001 C CNN
 F 3 "~" H 8050 7450 50  0001 C CNN
@@
 L Device:C C38
 U 1 1 5EFECEC2
-P 6550 7100
-F 0 "C38" H 6665 7146 50  0000 L CNN
-F 1 "C" H 6665 7055 50  0000 L CNN
-F 2 "Capacitor_SMD:C_0603_1608Metric" H 6588 6950 50  0001 C CNN
-F 3 "~" H 6550 7100 50  0001 C CNN
-	1    6550 7100
+P 6550 7150
+F 0 "C38" H 6665 7196 50  0000 L CNN
+F 1 ".1uF" H 6665 7105 50  0000 L CNN
+F 2 "Capacitor_SMD:C_0603_1608Metric" H 6588 7000 50  0001 C CNN
+F 3 "~" H 6550 7150 50  0001 C CNN
+	1    6550 7150
 	1    0    0    -1
 $EndComp
 Wire Wire Line
-	6550 7250 6300 7250
+	6550 7300 6300 7300
 Wire Wire Line
-	6550 7250 6800 7250
-Connection ~ 6550 7250
-Text GLabel 6800 7250 2    50   Input ~ 0
+	6550 7300 6800 7300
+Connection ~ 6550 7300
+Text GLabel 6800 7300 2    50   Input ~ 0
 VSS
 $Comp
 L power:GND #PWR0164
 U 1 1 5F075C11
-P 6300 7250
-F 0 "#PWR0164" H 6300 7000 50  0001 C CNN
-F 1 "GND" V 6305 7122 50  0000 R CNN
-F 2 "" H 6300 7250 50  0001 C CNN
-F 3 "" H 6300 7250 50  0001 C CNN
-	1    6300 7250
+P 6300 7300
+F 0 "#PWR0164" H 6300 7050 50  0001 C CNN
+F 1 "GND" V 6305 7172 50  0000 R CNN
+F 2 "" H 6300 7300 50  0001 C CNN
+F 3 "" H 6300 7300 50  0001 C CNN
+	1    6300 7300
 	0    1    1    0
 $EndComp
@@
 Wire Wire Line
 	6050 3400 6100 3400
+Text GLabel 8000 8900 2    50   Input ~ 0
+VSS
+Wire Wire Line
+	6450 4500 7050 4500
+Text GLabel 12250 6600 1    50   Input ~ 0
+PGND2
 $EndSCHEMATC

Commit message: basically an emergency backup, going to reroute my board
Parts:
- removed C23, C31, C45, C46, C48, C49: 22uF, Capacitor_SMD:C_0603_1608Metric, symbol Device:C
- C20, C21: value .1uF -> 1nF
- C24, C30: value C -> 1nF
- C28, C29: value C -> .012uF
- C47: value 22uF -> 33uF
- F1, F2: footprint Fuse:Fuse_Blade_Mini_directSolder -> 3557-2:Fuseholder_Blade_Mini_Keystone_3557-2
- J1, J4: footprint Connector_TE-Connectivity:TE_MATE-N-LOK_1-770866-x_1x02_P4.14mm_Vertical -> Connector_JST:JST_VH_B2PS-VH_1x02_P3.96mm_Horizontal
- L2, L3: footprint Inductor_SMD:L_Vishay_IHLP-2525 -> SRP7030-4R7M:SRP7030-4R7M
- R25: value R_US -> 5.36kOhm
- R26, R31: value R_US -> 40.2kOhm
- R27: value R_US -> 14kOhm
- R28: value 30Ohm -> 31Ohm
- R29: value R_US -> 9.31kOhm
- R30: value R_US -> 8.87kOhm
- R38, R41, R42: value R_US -> 5kOhm
Connections:
- net GNDREF: now also C47.2; no longer C47.1
- net Q4D: no longer C8.1, C9.1, IC1.1 (VIN), R39.2
- net SRN: now also C8.1, C9.1, IC1.1 (VIN), R39.2
- net at IC3.1 (VIN), L3.2, R43.2: now also C47.1; no longer C47.2
Other:
- moved on the sheet: C44, C47, C8, C9, CCD1, CIN1, CIN2, CVD1, F2, IC1, J2, Q6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

Commit message: Fixed CAN resistors and added filtering
Parts:
- added C? (x2): 1nF, Capacitor_SMD:C_0603_1608Metric, symbol Device:C
- added C? (x3): 100nF, Capacitor_SMD:C_0603_1608Metric, symbol Device:C
- added C?: 2.2uF, Capacitor_SMD:C_0603_1608Metric, symbol Device:C
- added L?: 2.2uH, Inductor_SMD:L_0603_1608Metric, symbol Device:L
- added R?: 3.3Ohm, Resistor_SMD:R_0603_1608Metric, symbol Device:R_US
- IC1, IC2, IC3: symbol FAN4010IL6X_F113:FAN4010IL6X_F113 -> Batteryboard-rescue:FAN4010IL6X_F113-FAN4010IL6X_F113
- NP1, NP2: value 120 -> 60
- TMP1: symbol MASA-LIB:LM50CIM3X -> Batteryboard-rescue:LM50CIM3X-MASA-LIB
- U2: symbol TPS65279DAPR:TPS65279DAPR -> Batteryboard-rescue:TPS65279DAPR-TPS65279DAPR
- U4: symbol PIC18F25K50-ISO:PIC18F25K50-I_SO -> Batteryboard-rescue:PIC18F25K50-I_SO-PIC18F25K50-ISO
Connections:
- wire segments 479 -> 494
Changed lines of the file:
@@
 FB2
 $Comp
-L FAN4010IL6X_F113:FAN4010IL6X_F113 IC2
+L Batteryboard-rescue:FAN4010IL6X_F113-FAN4010IL6X_F113 IC2
 U 1 1 5E16FEE4
 P 11250 9300
@@
 $EndComp
 $Comp
-L FAN4010IL6X_F113:FAN4010IL6X_F113 IC3
+L Batteryboard-rescue:FAN4010IL6X_F113-FAN4010IL6X_F113 IC3
 U 1 1 5E16B258
 P 15800 8550
@@
 Text GLabel 5000 8100 0    50   Input ~ 0
 TEMP_OUT
-$Comp
-L power:GND #PWR0166
-U 1 1 5F0B7350
-P 5000 9600
-F 0 "#PWR0166" H 5000 9350 50  0001 C CNN
-F 1 "GND" V 5005 9472 50  0000 R CNN
-F 2 "" H 5000 9600 50  0001 C CNN
-F 3 "" H 5000 9600 50  0001 C CNN
-	1    5000 9600
-	1    0    0    -1
-$EndComp
-$Comp
-L Device:C C34
-U 1 1 5F0B575C
-P 5000 9450
-F 0 "C34" V 5252 9450 50  0000 C CNN
-F 1 ".1uF" V 5161 9450 50  0000 C CNN
-F 2 "Capacitor_SMD:C_0603_1608Metric" H 5038 9300 50  0001 C CNN
-F 3 "~" H 5000 9450 50  0001 C CNN
-	1    5000 9450
-	-1   0    0    1
-$EndComp
 $Comp
 L power:GND #PWR0165
@@
 $EndComp
 $Comp
-L Device:R_US NP?
-U 1 1 5ED2EE3E
-P 4800 11550
-AR Path="/5ECB4406/5ED2EE3E" Ref="NP?"  Part="1"
-AR Path="/5ED2EE3E" Ref="NP2"  Part="1"
-F 0 "NP2" H 4868 11596 50  0000 L CNN
-F 1 "120" H 4868 11505 50  0000 L CNN
-F 2 "Resistor_SMD:R_0603_1608Metric" V 4840 11540 50  0001 C CNN
-F 3 "~" H 4800 11550 50  0001 C CNN
-	1    4800 11550
-	1    0    0    -1
-$EndComp
-$Comp
 L Device:C C?
 U 1 1 5ED2EE38
@@
 $EndComp
 $Comp
-L Device:R_US NP?
-U 1 1 5ED2EE1A
-P 4800 11150
-AR Path="/5ECB4406/5ED2EE1A" Ref="NP?"  Part="1"
-AR Path="/5ED2EE1A" Ref="NP1"  Part="1"
-F 0 "NP1" H 4868 11196 50  0000 L CNN
-F 1 "120" H 4868 11105 50  0000 L CNN
-F 2 "Resistor_SMD:R_0603_1608Metric" V 4840 11140 50  0001 C CNN
-F 3 "~" H 4800 11150 50  0001 C CNN
-	1    4800 11150
-	1    0    0    -1
-$EndComp
-$Comp
 L power:GND #PWR0139
 U 1 1 5E682ED3
@@
 	13650 9350 13550 9350
 Connection ~ 13200 9450
-Text GLabel 15400 9900 2    50   Input ~ 0
+Text GLabel 17050 9900 2    50   Input ~ 0
 TEMP_OUT
-Text GLabel 14600 9900 0    50   Input ~ 0
-5V0
 $Comp
 L power:GND #PWR0151
@@
 	12450 7900 12250 7900
 $Comp
-L TPS65279DAPR:TPS65279DAPR U2
+L Batteryboard-rescue:TPS65279DAPR-TPS65279DAPR U2
 U 1 1 5E217675
 P 12500 7000
@@
 	0    1    1    0
 $EndComp
-Text GLabel 13750 10050 2    50   Input ~ 0
+Text GLabel 13750 10050 3    50   Input ~ 0
 RLIM1
 Wire Wire Line
@@
 	12500 7800 12450 7800
 $Comp
-L MASA-LIB:LM50CIM3X TMP1
+L Batteryboard-rescue:LM50CIM3X-MASA-LIB TMP1
 U 1 1 5E0BF102
 P 15000 9900
@@
 PGC
 $Comp
-L PIC18F25K50-ISO:PIC18F25K50-I_SO U4
+L Batteryboard-rescue:PIC18F25K50-I_SO-PIC18F25K50-ISO U4
 U 1 1 5EEDA796
 P 5000 8000
@@
 7.4V LINE
 $Comp
-L FAN4010IL6X_F113:FAN4010IL6X_F113 IC1
+L Batteryboard-rescue:FAN4010IL6X_F113-FAN4010IL6X_F113 IC1
 U 1 1 5E171494
 P 10100 1650
@@
 Wire Wire Line
 	9300 4500 9700 4500
+Text GLabel 14200 9900 1    50   Input ~ 0
+5V0
+$Comp
+L Device:R_US NP?
+U 1 1 5ED2EE1A
+P 4800 11150
+AR Path="/5ECB4406/5ED2EE1A" Ref="NP?"  Part="1"
+AR Path="/5ED2EE1A" Ref="NP1"  Part="1"
+F 0 "NP1" H 4868 11196 50  0000 L CNN
+F 1 "60" H 4868 11105 50  0000 L CNN
+F 2 "Resistor_SMD:R_0603_1608Metric" V 4840 11140 50  0001 C CNN
+F 3 "~" H 4800 11150 50  0001 C CNN
+	1    4800 11150
+	1    0    0    -1
+$EndComp
+$Comp
+L Device:R_US NP?
+U 1 1 5ED2EE3E
+P 4800 11550
+AR Path="/5ECB4406/5ED2EE3E" Ref="NP?"  Part="1"
+AR Path="/5ED2EE3E" Ref="NP2"  Part="1"
+F 0 "NP2" H 4868 11596 50  0000 L CNN
+F 1 "60" H 4868 11505 50  0000 L CNN
+F 2 "Resistor_SMD:R_0603_1608Metric" V 4840 11540 50  0001 C CNN
+F 3 "~" H 4800 11550 50  0001 C CNN
+	1    4800 11550
+	1    0    0    -1
+$EndComp
+$Comp
+L power:GND #PWR0166
+U 1 1 5F0B7350
+P 5000 9600
+F 0 "#PWR0166" H 5000 9350 50  0001 C CNN
+F 1 "GND" V 5005 9472 50  0000 R CNN
+F 2 "" H 5000 9600 50  0001 C CNN
+F 3 "" H 5000 9600 50  0001 C CNN
+	1    5000 9600
+	1    0    0    -1
+$EndComp
+$Comp
+L Device:C C34
+U 1 1 5F0B575C
+P 5000 9450
+F 0 "C34" V 5252 9450 50  0000 C CNN
+F 1 ".1uF" V 5161 9450 50  0000 C CNN
+F 2 "Capacitor_SMD:C_0603_1608Metric" H 5038 9300 50  0001 C CNN
+F 3 "~" H 5000 9450 50  0001 C CNN
+	1    5000 9450
+	-1   0    0    1
+$EndComp
+$Comp
+L Device:C C?
+U 1 1 5E428FCB
+P 14200 10050
+F 0 "C?" V 13948 10050 50  0000 C CNN
+F 1 "1nF" V 14039 10050 50  0000 C CNN
+F 2 "Capacitor_SMD:C_0603_1608Metric" H 14238 9900 50  0001 C CNN
+F 3 "~" H 14200 10050 50  0001 C CNN
+	1    14200 10050
+	1    0    0    -1
+$EndComp
+$Comp
+L Device:C C?
+U 1 1 5E429589
+P 14400 10050
+F 0 "C?" V 14148 10050 50  0000 C CNN
+F 1 "100nF" V 14239 10050 50  0000 C CNN
+F 2 "Capacitor_SMD:C_0603_1608Metric" H 14438 9900 50  0001 C CNN
+F 3 "~" H 14400 10050 50  0001 C CNN
+	1    14400 10050
+	-1   0    0    1
+$EndComp
+Wire Wire Line
+	14200 9900 14400 9900
+Connection ~ 14400 9900
+Wire Wire Line
+	14400 9900 14600 9900
+Wire Wire Line
+	14400 10200 14300 10200
+$Comp
+L power:GND #PWR?
+U 1 1 5E499F7C
+P 14300 10200
+F 0 "#PWR?" H 14300 9950 50  0001 C CNN
+F 1 "GND" H 14305 10027 50  0000 C CNN
+F 2 "" H 14300 10200 50  0001 C CNN
+F 3 "" H 14300 10200 50  0001 C CNN
+	1    14300 10200
+	1    0    0    -1
+$EndComp
+Connection ~ 14300 10200
+Wire Wire Line
+	14300 10200 14200 10200
+$Comp
+L Device:C C?
+U 1 1 5E49A4E1
+P 15550 10050
+F 0 "C?" V 15298 10050 50  0000 C CNN
+F 1 "1nF" V 15389 10050 50  0000 C CNN
+F 2 "Capacitor_SMD:C_0603_1608Metric" H 15588 9900 50  0001 C CNN
+F 3 "~" H 15550 10050 50  0001 C CNN
+	1    15550 10050
+	-1   0    0    1
+$EndComp
+$Comp
+L Device:C C?
+U 1 1 5E49ACDA
+P 15950 10050
+F 0 "C?" V 15698 10050 50  0000 C CNN
+F 1 "100nF" V 15789 10050 50  0000 C CNN
+F 2 "Capacitor_SMD:C_0603_1608Metric" H 15988 9900 50  0001 C CNN
+F 3 "~" H 15950 10050 50  0001 C CNN
+	1    15950 10050
+	-1   0    0    1
+$EndComp
+$Comp
+L Device:C C?
+U 1 1 5E49AFF1
+P 16600 10050
+F 0 "C?" V 16348 10050 50  0000 C CNN
+F 1 "100nF" V 16439 10050 50  0000 C CNN
+F 2 "Capacitor_SMD:C_0603_1608Metric" H 16638 9900 50  0001 C CNN
+F 3 "~" H 16600 10050 50  0001 C CNN
+	1    16600 10050
+	-1   0    0    1
+$EndComp
+$Comp
+L Device:C C?
+U 1 1 5E49B600
+P 17050 10050
+F 0 "C?" V 16798 10050 50  0000 C CNN
+F 1 "2.2uF" V 16889 10050 50  0000 C CNN
+F 2 "Capacitor_SMD:C_0603_1608Metric" H 17088 9900 50  0001 C CNN
+F 3 "~" H 17050 10050 50  0001 C CNN
+	1    17050 10050
+	-1   0    0    1
+$EndComp
+$Comp
+L Device:R_US R?
+U 1 1 5E49BA5F
+P 16850 10300
+F 0 "R?" H 16918 10346 50  0000 L CNN
+F 1 "3.3Ohm" H 16918 10255 50  0000 L CNN
+F 2 "Resistor_SMD:R_0603_1608Metric" V 16890 10290 50  0001 C CNN
+F 3 "~" H 16850 10300 50  0001 C CNN
+	1    16850 10300
+	0    1    1    0
+$EndComp
+$Comp
+L Device:L L?
+U 1 1 5E49C1EF
+P 16300 9900
+F 0 "L?" V 16490 9900 50  0000 C CNN
+F 1 "2.2uH" V 16399 9900 50  0000 C CNN
+F 2 "Inductor_SMD:L_0603_1608Metric" H 16300 9900 50  0001 C CNN
+F 3 "~" H 16300 9900 50  0001 C CNN
+	1    16300 9900
+	0    -1   -1   0
+$EndComp
+Wire Wire Line
+	15400 9900 15550 9900
+Connection ~ 15550 9900
+Wire Wire Line
+	15550 9900 15950 9900
+Connection ~ 15950 9900
+Wire Wire Line
+	15950 9900 16150 9900
+Wire Wire Line
+	16450 9900 16600 9900
+Connection ~ 16600 9900
+Wire Wire Line
+	16600 9900 17050 9900
+Wire Wire Line
+	17050 10200 17050 10300
+Wire Wire Line
+	17050 10300 17000 10300
+Wire Wire Line
+	16700 10300 16600 10300
+Wire Wire Line
+	16600 10300 16600 10200
+Wire Wire Line
+	15950 10200 15750 10200
+$Comp
+L power:GND #PWR?
+U 1 1 5E5BCE71
+P 15750 10200
+F 0 "#PWR?" H 15750 9950 50  0001 C CNN
+F 1 "GND" H 15755 10027 50  0000 C CNN
+F 2 "" H 15750 10200 50  0001 C CNN
+F 3 "" H 15750 10200 50  0001 C CNN
+	1    15750 10200
+	1    0    0    -1
+$EndComp
+Connection ~ 15750 10200
+Wire Wire Line
+	15750 10200 15550 10200
+$Comp
+L power:GND #PWR?
+U 1 1 5E5BD350
+P 16600 10300
+F 0 "#PWR?" H 16600 10050 50  0001 C CNN
+F 1 "GND" H 16605 10127 50  0000 C CNN
+F 2 "" H 16600 10300 50  0001 C CNN
+F 3 "" H 16600 10300 50  0001 C CNN
+	1    16600 10300
+	1    0    0    -1
+$EndComp
+Connection ~ 16600 10300
 $EndSCHEMATC
