File: Batteryboard.sch (KiCad schematic (older format))
At the start: 164 parts, among them IC1 FAN4010IL6X_F113, IC2 FAN4010IL6X_F113, IC3 FAN4010IL6X_F113, J1 Conn_01x02_Male, J2 Conn_01x03_Male, J3 Conn_01x05_Male, J4 Conn_01x02_Male, J5 SC_19-20, J6 Conn_01x04_Male, Q1 SI7617DN-T1-GE3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

Commit message: fixed stuff
Parts:
- removed J5: SC_19-20, MASA-LIB:bottom_Stack_Connector_2019_2020, symbol Batteryboard-rescue:SC_19-20-MASA-LIB
- added J7: SC_19-20, MASA_Library:Stack_Connector_2019_2020, symbol MASA-LIB:SC_19-20
Connections:
- net 3V3: now also J7.2 (3V3), J7.3 (3V3), J7.6 (3V3), J7.7 (3V3)
- net 5V0: now also J7.34 (5V0), J7.35 (5V0), J7.38 (5V0), J7.39 (5V0)
- net CAN_H: now also J7.21 (CAN_H)
- net CAN_L: now also J7.23 (CAN_L)
- net GND: now also J7.1 (GND), J7.19 (GND), J7.20 (GND), J7.36 (GND), J7.37 (GND), J7.4 (GND), J7.40 (GND), J7.5 (GND)
- net UART1_RX: now also J7.27 (UART1_RX)
- net UART1_TX: now also J7.25 (UART1_TX)
Changed lines of the file:
@@
-$EndComp
-$Comp
-L Batteryboard-rescue:SC_19-20-MASA-LIB J5
-U 1 1 5E021180
-P 1900 7150
-F 0 "J5" H 1900 7315 50  0000 C CNN
-F 1 "SC_19-20" H 1900 7224 50  0000 C CNN
-F 2 "MASA-LIB:bottom_Stack_Connector_2019_2020" H 1650 7300 50  0001 L CNN
-F 3 "" H 1650 7800 50  0001 L CNN
-F 4 "Conn Shrouded Header HDR 40 POS 1.27mm Solder ST SMD T/R" H 1650 7700 50  0001 L CNN "Description"
-F 5 "11.35" H 1650 7500 50  0001 L CNN "Height"
-F 6 "SAMTEC" H 1650 7400 50  0001 L CNN "Manufacturer_Name"
-F 7 "TFC-120-32-F-D-A-K-TR" H 1650 7600 50  0001 L CNN "Manufacturer_Part_Number"
-	1    1900 7150
-	1    0    0    -1
 $EndComp
 $Comp
@@
 Wire Wire Line
 	12700 4350 12450 4350
+$Comp
+L MASA-LIB:SC_19-20 J7
+U 1 1 5E686151
+P 1900 7150
+F 0 "J7" H 1900 7315 50  0000 C CNN
+F 1 "SC_19-20" H 1900 7224 50  0000 C CNN
+F 2 "MASA_Library:Stack_Connector_2019_2020" H 1650 7300 50  0001 L CNN
+F 3 "" H 1650 7800 50  0001 L CNN
+F 4 "Conn Shrouded Header HDR 40 POS 1.27mm Solder ST SMD T/R" H 1650 7700 50  0001 L CNN "Description"
+F 5 "11.35" H 1650 7500 50  0001 L CNN "Height"
+F 6 "SAMTEC" H 1650 7400 50  0001 L CNN "Manufacturer_Name"
+F 7 "TFC-120-32-F-D-A-K-TR" H 1650 7600 50  0001 L CNN "Manufacturer_Part_Number"
+	1    1900 7150
+	1    0    0    -1
+$EndComp
 $EndSCHEMATC

Commit message: fixed some shit
Connections:
- net GND: no longer J7.1 (GND), J7.19 (GND), J7.20 (GND), J7.36 (GND), J7.37 (GND), J7.4 (GND), J7.40 (GND), J7.5 (GND)
- net GNDREF: now also J7.1 (GND), J7.19 (GND), J7.20 (GND), J7.36 (GND), J7.37 (GND), J7.4 (GND), J7.40 (GND), J7.5 (GND)
Changed lines of the file:
@@
 	1    0    0    -1
-$EndComp
-$Comp
-L power:GND #PWR0133
-U 1 1 5E02CE50
-P 2550 8950
-F 0 "#PWR0133" H 2550 8700 50  0001 C CNN
-F 1 "GND" V 2555 8822 50  0000 R CNN
-F 2 "" H 2550 8950 50  0001 C CNN
-F 3 "" H 2550 8950 50  0001 C CNN
-	1    2550 8950
-	0    -1   -1   0
-$EndComp
-$Comp
-L power:GND #PWR0132
-U 1 1 5E02D39E
-P 2550 9150
-F 0 "#PWR0132" H 2550 8900 50  0001 C CNN
-F 1 "GND" V 2555 9022 50  0000 R CNN
-F 2 "" H 2550 9150 50  0001 C CNN
-F 3 "" H 2550 9150 50  0001 C CNN
-	1    2550 9150
-	0    -1   -1   0
-$EndComp
-$Comp
-L power:GND #PWR0131
-U 1 1 5E02EC52
-P 2550 8150
-F 0 "#PWR0131" H 2550 7900 50  0001 C CNN
-F 1 "GND" V 2555 8022 50  0000 R CNN
-F 2 "" H 2550 8150 50  0001 C CNN
-F 3 "" H 2550 8150 50  0001 C CNN
-	1    2550 8150
-	0    -1   -1   0
 $EndComp
 Text GLabel 2550 7450 2    50   Input ~ 0
@@
 Text GLabel 2550 8850 2    50   Input ~ 0
 5V0
-$Comp
-L power:GND #PWR0130
-U 1 1 5E038DA8
-P 1250 8150
-F 0 "#PWR0130" H 1250 7900 50  0001 C CNN
-F 1 "GND" V 1255 8022 50  0000 R CNN
-F 2 "" H 1250 8150 50  0001 C CNN
-F 3 "" H 1250 8150 50  0001 C CNN
-	1    1250 8150
-	0    1    1    0
-$EndComp
 Text GLabel 1250 8550 0    50   Input ~ 0
 UART1_RX
@@
 3V3
 $Comp
-L power:GND #PWR0129
-U 1 1 5E02F0D8
-P 2550 7350
-F 0 "#PWR0129" H 2550 7100 50  0001 C CNN
-F 1 "GND" V 2555 7222 50  0000 R CNN
-F 2 "" H 2550 7350 50  0001 C CNN
-F 3 "" H 2550 7350 50  0001 C CNN
-	1    2550 7350
-	0    -1   -1   0
-$EndComp
-$Comp
-L power:GND #PWR0128
-U 1 1 5E02B2BE
-P 1250 9050
-F 0 "#PWR0128" H 1250 8800 50  0001 C CNN
-F 1 "GND" V 1255 8922 50  0000 R CNN
-F 2 "" H 1250 9050 50  0001 C CNN
-F 3 "" H 1250 9050 50  0001 C CNN
-	1    1250 9050
-	0    1    1    0
-$EndComp
-$Comp
-L power:GND #PWR0127
-U 1 1 5E02737A
-P 1250 7450
-F 0 "#PWR0127" H 1250 7200 50  0001 C CNN
-F 1 "GND" V 1255 7322 50  0000 R CNN
-F 2 "" H 1250 7450 50  0001 C CNN
-F 3 "" H 1250 7450 50  0001 C CNN
-	1    1250 7450
-	0    1    1    0
-$EndComp
-$Comp
-L power:GND #PWR0124
-U 1 1 5E023948
-P 1250 7250
-F 0 "#PWR0124" H 1250 7000 50  0001 C CNN
-F 1 "GND" V 1255 7122 50  0000 R CNN
-F 2 "" H 1250 7250 50  0001 C CNN
-F 3 "" H 1250 7250 50  0001 C CNN
-	1    1250 7250
-	0    1    1    0
-$EndComp
-$Comp
 L Connector:Conn_01x05_Male J3
 U 1 1 5E1B735E
@@
 	1    0    0    -1
 $EndComp
+$Comp
+L power:GNDREF #PWR0124
+U 1 1 5E889489
+P 1250 7250
+F 0 "#PWR0124" H 1250 7000 50  0001 C CNN
+F 1 "GNDREF" V 1255 7122 50  0000 R CNN
+F 2 "" H 1250 7250 50  0001 C CNN
+F 3 "" H 1250 7250 50  0001 C CNN
+	1    1250 7250
+	0    1    1    0
+$EndComp
+$Comp
+L power:GNDREF #PWR0127
+U 1 1 5E88C1F5
+P 1250 7450
+F 0 "#PWR0127" H 1250 7200 50  0001 C CNN
+F 1 "GNDREF" V 1255 7322 50  0000 R CNN
+F 2 "" H 1250 7450 50  0001 C CNN
+F 3 "" H 1250 7450 50  0001 C CNN
+	1    1250 7450
+	0    1    1    0
+$EndComp
+$Comp
+L power:GNDREF #PWR0128
+U 1 1 5E88DA65
+P 2550 7350
+F 0 "#PWR0128" H 2550 7100 50  0001 C CNN
+F 1 "GNDREF" V 2555 7222 50  0000 R CNN
+F 2 "" H 2550 7350 50  0001 C CNN
+F 3 "" H 2550 7350 50  0001 C CNN
+	1    2550 7350
+	0    -1   -1   0
+$EndComp
+$Comp
+L power:GNDREF #PWR0129
+U 1 1 5E88F4E0
+P 1250 8150
+F 0 "#PWR0129" H 1250 7900 50  0001 C CNN
+F 1 "GNDREF" V 1255 8022 50  0000 R CNN
+F 2 "" H 1250 8150 50  0001 C CNN
+F 3 "" H 1250 8150 50  0001 C CNN
+	1    1250 8150
+	0    1    1    0
+$EndComp
+$Comp
+L power:GNDREF #PWR0130
+U 1 1 5E890BF1
+P 2550 8150
+F 0 "#PWR0130" H 2550 7900 50  0001 C CNN
+F 1 "GNDREF" V 2555 8022 50  0000 R CNN
+F 2 "" H 2550 8150 50  0001 C CNN
+F 3 "" H 2550 8150 50  0001 C CNN
+	1    2550 8150
+	0    -1   -1   0
+$EndComp
+$Comp
+L power:GNDREF #PWR0131
+U 1 1 5E8911D4
+P 2550 8950
+F 0 "#PWR0131" H 2550 8700 50  0001 C CNN
+F 1 "GNDREF" V 2555 8822 50  0000 R CNN
+F 2 "" H 2550 8950 50  0001 C CNN
+F 3 "" H 2550 8950 50  0001 C CNN
+	1    2550 8950
+	0    -1   -1   0
+$EndComp
+$Comp
+L power:GNDREF #PWR0132
+U 1 1 5E894637
+P 2550 9150
+F 0 "#PWR0132" H 2550 8900 50  0001 C CNN
+F 1 "GNDREF" V 2555 9022 50  0000 R CNN
+F 2 "" H 2550 9150 50  0001 C CNN
+F 3 "" H 2550 9150 50  0001 C CNN
+	1    2550 9150
+	0    -1   -1   0
+$EndComp
+$Comp
+L power:GNDREF #PWR0133
+U 1 1 5E8960A2
+P 1250 9050
+F 0 "#PWR0133" H 1250 8800 50  0001 C CNN
+F 1 "GNDREF" V 1255 8922 50  0000 R CNN
+F 2 "" H 1250 9050 50  0001 C CNN
+F 3 "" H 1250 9050 50  0001 C CNN
+	1    1250 9050
+	0    1    1    0
+$EndComp
 $EndSCHEMATC
